File: hw/bridge/can.kicad_sch (KiCad schematic)
At the start: 4 parts, among them U5 TJA1051T-3

Commit message: Add initial PCB to the bridge
Signed-off-by: Mateusz Pająk <22417805+Tai-Min@users.noreply.github.com>
Parts:
- C11, C12: footprint (none) -> Capacitor_SMD:C_1206_3216Metric
- R6: footprint (none) -> Resistor_SMD:R_1206_3216Metric
Changed lines of the file:
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@@
 			)
 		)
-		(property "Footprint" ""
+		(property "Footprint" "Capacitor_SMD:C_1206_3216Metric"
 			(at 171.7548 72.39 0)
 			(effects
@@
 			)
 		)
-		(property "Footprint" ""
+		(property "Footprint" "Resistor_SMD:R_1206_3216Metric"
 			(at 177.292 102.87 90)
 			(effects
@@
 			)
 		)
-		(property "Footprint" ""
+		(property "Footprint" "Capacitor_SMD:C_1206_3216Metric"
 			(at 161.5948 72.39 0)
 			(effects

Commit message: Fix jumpers
Signed-off-by: Mateusz Pająk <22417805+Tai-Min@users.noreply.github.com>
Parts:
- renumbered R6 to R13, U5 to U6
Changed lines of the file:
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@@
 		(on_board yes)
 		(dnp no)
-		(property "Reference" "#PWR036"
+		(property "Reference" "#PWR050"
 			(at 172.72 87.63 0)
 			(effects
@@
 			(project "bridge"
 				(path "/3b0cc3d4-df75-4145-abb6-d19d57c31f1b/4c6f2595-f15e-4244-9b90-548609f15b3d"
-					(reference "#PWR036")
+					(reference "#PWR050")
 					(unit 1)
 				)
@@
 		(dnp no)
 		(fields_autoplaced yes)
-		(property "Reference" "#PWR032"
+		(property "Reference" "#PWR049"
 			(at 172.72 74.93 0)
 			(effects
@@
 			(project "bridge"
 				(path "/3b0cc3d4-df75-4145-abb6-d19d57c31f1b/4c6f2595-f15e-4244-9b90-548609f15b3d"
-					(reference "#PWR032")
+					(reference "#PWR049")
 					(unit 1)
 				)
@@
 		(on_board yes)
 		(dnp no)
-		(property "Reference" "#PWR037"
+		(property "Reference" "#PWR044"
 			(at 137.16 107.95 0)
 			(effects
@@
 			(project "bridge"
 				(path "/3b0cc3d4-df75-4145-abb6-d19d57c31f1b/4c6f2595-f15e-4244-9b90-548609f15b3d"
-					(reference "#PWR037")
+					(reference "#PWR044")
 					(unit 1)
 				)
@@
 		(dnp no)
 		(fields_autoplaced yes)
-		(property "Reference" "#PWR033"
+		(property "Reference" "#PWR047"
 			(at 162.56 74.93 0)
 			(effects
@@
 			(project "bridge"
 				(path "/3b0cc3d4-df75-4145-abb6-d19d57c31f1b/4c6f2595-f15e-4244-9b90-548609f15b3d"
-					(reference "#PWR033")
+					(reference "#PWR047")
 					(unit 1)
 				)
@@
 		(on_board yes)
 		(dnp no)
-		(property "Reference" "#PWR039"
+		(property "Reference" "#PWR046"
 			(at 153.67 121.92 0)
 			(effects
@@
 			(project "bridge"
 				(path "/3b0cc3d4-df75-4145-abb6-d19d57c31f1b/4c6f2595-f15e-4244-9b90-548609f15b3d"
-					(reference "#PWR039")
+					(reference "#PWR046")
 					(unit 1)
 				)
@@
 		(dnp no)
 		(fields_autoplaced yes)
-		(property "Reference" "#PWR035"
+		(property "Reference" "#PWR045"
 			(at 153.67 93.98 0)
 			(effects
@@
 			(project "bridge"
 				(path "/3b0cc3d4-df75-4145-abb6-d19d57c31f1b/4c6f2595-f15e-4244-9b90-548609f15b3d"
-					(reference "#PWR035")
+					(reference "#PWR045")
 					(unit 1)
 				)
@@
 		(dnp yes)
 		(fields_autoplaced yes)
-		(property "Reference" "R6"
+		(property "Reference" "R13"
 			(at 181.61 101.5999 0)
 			(effects
@@
 			(project ""
 				(path "/3b0cc3d4-df75-4145-abb6-d19d57c31f1b/4c6f2595-f15e-4244-9b90-548609f15b3d"
-					(reference "R6")
+					(reference "R13")
 					(unit 1)
 				)
@@
 		(on_board yes)
 		(dnp no)
-		(property "Reference" "#PWR034"
+		(property "Reference" "#PWR048"
 			(at 162.56 87.63 0)
 			(effects
@@
 			(project "bridge"
 				(path "/3b0cc3d4-df75-4145-abb6-d19d57c31f1b/4c6f2595-f15e-4244-9b90-548609f15b3d"
-					(reference "#PWR034")
+					(reference "#PWR048")
 					(unit 1)
 				)
@@
 		(dnp no)
 		(fields_autoplaced yes)
-		(property "Reference" "U5"
+		(property "Reference" "U6"
 			(at 155.8133 90.17 0)
 			(effects
@@
 			(project ""
 				(path "/3b0cc3d4-df75-4145-abb6-d19d57c31f1b/4c6f2595-f15e-4244-9b90-548609f15b3d"
-					(reference "U5")
-					(unit 1)
-				)
+					(reference "U6")
+					(unit 1)
+				)
