File: hw/bridge/pwr.kicad_sch (KiCad schematic)
At the start: 3 parts, among them U4 MCP1754S-3302xCB

Commit message: Add initial PCB to the bridge
Signed-off-by: Mateusz Pająk <22417805+Tai-Min@users.noreply.github.com>
Parts:
- C10, C9: footprint (none) -> Capacitor_SMD:C_1206_3216Metric
Changed lines of the file:
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@@
 			)
 		)
-		(property "Footprint" ""
+		(property "Footprint" "Capacitor_SMD:C_1206_3216Metric"
 			(at 138.7348 101.6 0)
 			(effects
@@
 			)
 		)
-		(property "Footprint" ""
+		(property "Footprint" "Capacitor_SMD:C_1206_3216Metric"
 			(at 175.5648 101.6 0)
 			(effects

Commit message: Fix jumpers
Signed-off-by: Mateusz Pająk <22417805+Tai-Min@users.noreply.github.com>
Parts:
- renumbered U4 to U5
Changed lines of the file:
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@@
 		(dnp no)
 		(fields_autoplaced yes)
-		(property "Reference" "#PWR031"
+		(property "Reference" "#PWR043"
 			(at 179.07 102.87 0)
 			(effects
@@
 			(project ""
 				(path "/3b0cc3d4-df75-4145-abb6-d19d57c31f1b/bdf538a0-d28a-4d8b-85d4-59a1db2dafb5"
-					(reference "#PWR031")
+					(reference "#PWR043")
 					(unit 1)
 				)
@@
 		(dnp no)
 		(fields_autoplaced yes)
-		(property "Reference" "#PWR030"
+		(property "Reference" "#PWR042"
 			(at 156.21 118.11 0)
 			(effects
@@
 			(project "bridge"
 				(path "/3b0cc3d4-df75-4145-abb6-d19d57c31f1b/bdf538a0-d28a-4d8b-85d4-59a1db2dafb5"
-					(reference "#PWR030")
+					(reference "#PWR042")
 					(unit 1)
 				)
@@
 		(dnp no)
 		(fields_autoplaced yes)
-		(property "Reference" "U4"
+		(property "Reference" "U5"
 			(at 156.21 93.98 0)
 			(effects
@@
 			(project ""
 				(path "/3b0cc3d4-df75-4145-abb6-d19d57c31f1b/bdf538a0-d28a-4d8b-85d4-59a1db2dafb5"
-					(reference "U4")
+					(reference "U5")
 					(unit 1)
 				)
@@
 		(dnp no)
 		(fields_autoplaced yes)
-		(property "Reference" "#PWR011"
+		(property "Reference" "#PWR041"
 			(at 137.16 102.87 0)
 			(effects
@@
 			(project "bridge"
 				(path "/3b0cc3d4-df75-4145-abb6-d19d57c31f1b/bdf538a0-d28a-4d8b-85d4-59a1db2dafb5"
-					(reference "#PWR011")
-					(unit 1)
-				)
+					(reference "#PWR041")
+					(unit 1)
+				)
