File: hw/bridge/mcu.kicad_sch (KiCad schematic)
At the start: 10 parts, among them J4 SWD, J5 BOOT, U1 STM32G0B1CBT, Y1 8MHz

Commit message: Add initial PCB to the bridge
Signed-off-by: Mateusz Pająk <22417805+Tai-Min@users.noreply.github.com>
Parts:
- C4, C5, C6, C7, C8: footprint (none) -> Capacitor_SMD:C_1206_3216Metric
- J4: footprint (none) -> Connector_PinHeader_2.54mm:PinHeader_2x03_P2.54mm_Vertical
- J5: footprint (none) -> Connector_PinHeader_2.54mm:PinHeader_1x02_P2.54mm_Vertical
- R5: footprint (none) -> Resistor_SMD:R_1206_3216Metric
- Y1: value 8MHz -> HCI XC53G2-8.000-F12NJHP; footprint (none) -> Crystal:Crystal_SMD_5032-2Pin_5.0x3.2mm
Changed lines of the file:
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@@
 		(dnp no)
 		(property "Reference" "Y1"
-			(at 109.22 74.93 0)
-			(effects
-				(font
-					(size 1.27 1.27)
-				)
-			)
-		)
-		(property "Value" "8MHz"
-			(at 109.22 77.47 0)
-			(effects
-				(font
-					(size 1.27 1.27)
-				)
-			)
-		)
-		(property "Footprint" ""
+			(at 108.966 67.056 0)
+			(effects
+				(font
+					(size 1.27 1.27)
+				)
+			)
+		)
+		(property "Value" "HCI XC53G2-8.000-F12NJHP"
+			(at 109.22 64.516 0)
+			(effects
+				(font
+					(size 1.27 1.27)
+				)
+			)
+		)
+		(property "Footprint" "Crystal:Crystal_SMD_5032-2Pin_5.0x3.2mm"
 			(at 109.22 71.12 0)
 			(effects
@@
 			)
 		)
-		(property "Footprint" ""
+		(property "Footprint" "Capacitor_SMD:C_1206_3216Metric"
 			(at 90.4748 69.85 0)
 			(effects
@@
 			)
 		)
-		(property "Footprint" ""
+		(property "Footprint" "Capacitor_SMD:C_1206_3216Metric"
 			(at 101.9048 72.39 0)
 			(effects
@@
 			)
 		)
-		(property "Footprint" ""
+		(property "Footprint" "Connector_PinHeader_2.54mm:PinHeader_2x03_P2.54mm_Vertical"
 			(at 100.33 106.68 0)
 			(effects
@@
 			)
 		)
-		(property "Footprint" ""
+		(property "Footprint" "Capacitor_SMD:C_1206_3216Metric"
 			(at 151.4348 39.37 0)
 			(effects
@@
 			)
 		)
-		(property "Footprint" ""
+		(property "Footprint" "Resistor_SMD:R_1206_3216Metric"
 			(at 97.282 134.62 90)
 			(effects
@@
 			)
 		)
-		(property "Footprint" ""
+		(property "Footprint" "Connector_PinHeader_2.54mm:PinHeader_1x02_P2.54mm_Vertical"
 			(at 105.41 127 0)
 			(effects
@@
 			)
 		)
-		(property "Footprint" ""
+		(property "Footprint" "Capacitor_SMD:C_1206_3216Metric"
 			(at 114.6048 72.39 0)
 			(effects
@@
 			)
 		)
-		(property "Footprint" ""
+		(property "Footprint" "Capacitor_SMD:C_1206_3216Metric"
 			(at 141.2748 39.37 0)
 			(effects

Commit message: Fix jumpers
Signed-off-by: Mateusz Pająk <22417805+Tai-Min@users.noreply.github.com>
Parts:
- renumbered C6 to C4, C7 to C5, C8 to C6, C4 to C7, C5 to C8, R5 to R12, U1 to U4
Changed lines of the file:
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@@
 		(dnp no)
 		(fields_autoplaced yes)
-		(property "Reference" "#PWR028"
+		(property "Reference" "#PWR029"
 			(at 91.44 85.09 0)
 			(effects
@@
 			(project "bridge"
 				(path "/3b0cc3d4-df75-4145-abb6-d19d57c31f1b/ee32e54e-8e22-4372-9897-0863eef95f76"
-					(reference "#PWR028")
+					(reference "#PWR029")
 					(unit 1)
 				)
@@
 		(dnp no)
 		(fields_autoplaced yes)
-		(property "Reference" "#PWR027"
+		(property "Reference" "#PWR034"
 			(at 132.08 63.5 0)
 			(effects
@@
 			(project "bridge"
 				(path "/3b0cc3d4-df75-4145-abb6-d19d57c31f1b/ee32e54e-8e22-4372-9897-0863eef95f76"
-					(reference "#PWR027")
+					(reference "#PWR034")
 					(unit 1)
 				)
@@
 		(on_board yes)
 		(dnp no)
-		(property "Reference" "C6"
+		(property "Reference" "C4"
 			(at 85.598 72.898 90)
 			(effects
@@
 			(project "bridge"
 				(path "/3b0cc3d4-df75-4145-abb6-d19d57c31f1b/ee32e54e-8e22-4372-9897-0863eef95f76"
-					(reference "C6")
+					(reference "C4")
 					(unit 1)
 				)
@@
 		(on_board yes)
 		(dnp no)
-		(property "Reference" "C7"
+		(property "Reference" "C5"
 			(at 97.028 75.438 90)
 			(effects
@@
 			(project "bridge"
 				(path "/3b0cc3d4-df75-4145-abb6-d19d57c31f1b/ee32e54e-8e22-4372-9897-0863eef95f76"
-					(reference "C7")
+					(reference "C5")
 					(unit 1)
 				)
@@
 		(on_board yes)
 		(dnp no)
-		(property "Reference" "#PWR024"
+		(property "Reference" "#PWR038"
 			(at 152.4 54.61 0)
 			(effects
@@
 			(project "bridge"
 				(path "/3b0cc3d4-df75-4145-abb6-d19d57c31f1b/ee32e54e-8e22-4372-9897-0863eef95f76"
-					(reference "#PWR024")
+					(reference "#PWR038")
 					(unit 1)
 				)
@@
 		(dnp no)
 		(fields_autoplaced yes)
-		(property "Reference" "#PWR029"
+		(property "Reference" "#PWR033"
 			(at 109.22 88.9 0)
 			(effects
@@
 			(project "bridge"
 				(path "/3b0cc3d4-df75-4145-abb6-d19d57c31f1b/ee32e54e-8e22-4372-9897-0863eef95f76"
-					(reference "#PWR029")
+					(reference "#PWR033")
 					(unit 1)
 				)
@@
 		(on_board yes)
 		(dnp no)
-		(property "Reference" "#PWR022"
+		(property "Reference" "#PWR036"
 			(at 142.24 54.61 0)
 			(effects
@@
 			(project "bridge"
 				(path "/3b0cc3d4-df75-4145-abb6-d19d57c31f1b/ee32e54e-8e22-4372-9897-0863eef95f76"
-					(reference "#PWR022")
+					(reference "#PWR036")
 					(unit 1)
 				)
@@
 		(dnp no)
 		(fields_autoplaced yes)
-		(property "Reference" "#PWR019"
+		(property "Reference" "#PWR031"
 			(at 99.06 129.54 0)
 			(effects
@@
 			(project "bridge"
 				(path "/3b0cc3d4-df75-4145-abb6-d19d57c31f1b/ee32e54e-8e22-4372-9897-0863eef95f76"
-					(reference "#PWR019")
+					(reference "#PWR031")
 					(unit 1)
 				)
@@
 		(on_board yes)
 		(dnp no)
-		(property "Reference" "U1"
+		(property "Reference" "U4"
 			(at 164.592 149.352 0)
 			(effects
@@
 			(project "bridge"
 				(path "/3b0cc3d4-df75-4145-abb6-d19d57c31f1b/ee32e54e-8e22-4372-9897-0863eef95f76"
-					(reference "U1")
+					(reference "U4")
 					(unit 1)
 				)
@@
 		(dnp no)
 		(fields_autoplaced yes)
-		(property "Reference" "#PWR021"
+		(property "Reference" "#PWR035"
 			(at 142.24 41.91 0)
 			(effects
@@
 			(project "bridge"
 				(path "/3b0cc3d4-df75-4145-abb6-d19d57c31f1b/ee32e54e-8e22-4372-9897-0863eef95f76"
-					(reference "#PWR021")
+					(reference "#PWR035")
 					(unit 1)
 				)
@@
 		(on_board yes)
 		(dnp no)
-		(property "Reference" "C5"
+		(property "Reference" "C8"
 			(at 146.558 42.418 90)
 			(effects
@@
 			(project "bridge"
 				(path "/3b0cc3d4-df75-4145-abb6-d19d57c31f1b/ee32e54e-8e22-4372-9897-0863eef95f76"
-					(reference "C5")
+					(reference "C8")
 					(unit 1)
 				)
@@
 		(dnp no)
 		(fields_autoplaced yes)
-		(property "Reference" "#PWR018"
+		(property "Reference" "#PWR028"
 			(at 83.82 114.3 0)
 			(effects
@@
 			(project ""
 				(path "/3b0cc3d4-df75-4145-abb6-d19d57c31f1b/ee32e54e-8e22-4372-9897-0863eef95f76"
-					(reference "#PWR018")
+					(reference "#PWR028")
 					(unit 1)
 				)
@@
 		(dnp no)
 		(fields_autoplaced yes)
-		(property "Reference" "#PWR026"
+		(property "Reference" "#PWR040"
 			(at 162.56 54.61 0)
 			(effects
@@
 			(project "bridge"
 				(path "/3b0cc3d4-df75-4145-abb6-d19d57c31f1b/ee32e54e-8e22-4372-9897-0863eef95f76"
-					(reference "#PWR026")
+					(reference "#PWR040")
 					(unit 1)
 				)
@@
 		(dnp no)
 		(fields_autoplaced yes)
-		(property "Reference" "#PWR023"
+		(property "Reference" "#PWR037"
 			(at 152.4 41.91 0)
 			(effects
@@
 			(project "bridge"
 				(path "/3b0cc3d4-df75-4145-abb6-d19d57c31f1b/ee32e54e-8e22-4372-9897-0863eef95f76"
-					(reference "#PWR023")
+					(reference "#PWR037")
 					(unit 1)
 				)
@@
 		(dnp no)
 		(fields_autoplaced yes)
-		(property "Reference" "#PWR025"
+		(property "Reference" "#PWR039"
 			(at 161.29 157.48 0)
 			(effects
@@
 			(project "bridge"
 				(path "/3b0cc3d4-df75-4145-abb6-d19d57c31f1b/ee32e54e-8e22-4372-9897-0863eef95f76"
-					(reference "#PWR025")
+					(reference "#PWR039")
 					(unit 1)
 				)
@@
 		(dnp no)
 		(fields_autoplaced yes)
-		(property "Reference" "R5"
+		(property "Reference" "R12"
 			(at 101.6 133.3499 0)
 			(effects
@@
 			(project ""
 				(path "/3b0cc3d4-df75-4145-abb6-d19d57c31f1b/ee32e54e-8e22-4372-9897-0863eef95f76"
-					(reference "R5")
+					(reference "R12")
 					(unit 1)
 				)
@@
 		(on_board yes)
 		(dnp no)
-		(property "Reference" "C8"
+		(property "Reference" "C6"
 			(at 119.126 74.93 90)
 			(effects
@@
 			(project "bridge"
 				(path "/3b0cc3d4-df75-4145-abb6-d19d57c31f1b/ee32e54e-8e22-4372-9897-0863eef95f76"
-					(reference "C8")
+					(reference "C6")
 					(unit 1)
 				)
@@
 		(dnp no)
 		(fields_autoplaced yes)
-		(property "Reference" "#PWR017"
+		(property "Reference" "#PWR030"
 			(at 92.71 105.41 0)
 			(effects
@@
 			(project ""
 				(path "/3b0cc3d4-df75-4145-abb6-d19d57c31f1b/ee32e54e-8e22-4372-9897-0863eef95f76"
-					(reference "#PWR017")
+					(reference "#PWR030")
 					(unit 1)
 				)
@@
 		(on_board yes)
 		(dnp no)
-		(property "Reference" "C4"
+		(property "Reference" "C7"
 			(at 136.398 42.418 90)
 			(effects
@@
 			(project "bridge"
 				(path "/3b0cc3d4-df75-4145-abb6-d19d57c31f1b/ee32e54e-8e22-4372-9897-0863eef95f76"
-					(reference "C4")
+					(reference "C7")
 					(unit 1)
 				)
@@
 		(dnp no)
 		(fields_autoplaced yes)
-		(property "Reference" "#PWR020"
+		(property "Reference" "#PWR032"
 			(at 99.06 146.05 0)
 			(effects
@@
 			(project "bridge"
 				(path "/3b0cc3d4-df75-4145-abb6-d19d57c31f1b/ee32e54e-8e22-4372-9897-0863eef95f76"
-					(reference "#PWR020")
-					(unit 1)
-				)
+					(reference "#PWR032")
+					(unit 1)
+				)

Commit message: Redesign the PCB, remove DNP components
Signed-off-by: Mateusz Pająk <22417805+Tai-Min@users.noreply.github.com>
Parts:
- C4: value 100n / 50V -> 100n / 16V; footprint Capacitor_SMD:C_1206_3216Metric -> Capacitor_SMD:C_0603_1608Metric
- C5, C7, C8: footprint Capacitor_SMD:C_1206_3216Metric -> Capacitor_SMD:C_0603_1608Metric
- C6: value 6p / 50V -> 6p / 16V; footprint Capacitor_SMD:C_1206_3216Metric -> Capacitor_SMD:C_0603_1608Metric
- R12: footprint Resistor_SMD:R_1206_3216Metric -> Resistor_SMD:R_0603_1608Metric
Other:
- note added: "8MHz"
Changed lines of the file:
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@@
 	(generator_version "9.0")
 	(paper "A4")
+	(text "8MHz"
+		(exclude_from_sim no)
+		(at 109.22 75.184 0)
+		(effects
+			(font
+				(size 1.27 1.27)
+			)
+		)
+	)
 	(text "VREF/VDD"
 		(exclude_from_sim no)
@@
 			)
 		)
-		(property "Value" "100n / 50V"
+		(property "Value" "100n / 16V"
 			(at 87.63 71.6281 90)
 			(effects
@@
 			)
 		)
-		(property "Footprint" "Capacitor_SMD:C_1206_3216Metric"
+		(property "Footprint" "Capacitor_SMD:C_0603_1608Metric"
 			(at 90.4748 69.85 0)
 			(effects
@@
 			)
 		)
-		(property "Footprint" "Capacitor_SMD:C_1206_3216Metric"
+		(property "Footprint" "Capacitor_SMD:C_0603_1608Metric"
 			(at 101.9048 72.39 0)
 			(effects
@@
 			)
 		)
-		(property "Footprint" "Capacitor_SMD:C_1206_3216Metric"
+		(property "Footprint" "Capacitor_SMD:C_0603_1608Metric"
 			(at 151.4348 39.37 0)
 			(effects
@@
 			)
 		)
-		(property "Footprint" "Resistor_SMD:R_1206_3216Metric"
+		(property "Footprint" "Resistor_SMD:R_0603_1608Metric"
 			(at 97.282 134.62 90)
 			(effects
@@
 			)
 		)
-		(property "Value" "6p / 50V"
+		(property "Value" "6p / 16V"
 			(at 121.158 73.6601 90)
 			(effects
@@
 			)
 		)
-		(property "Footprint" "Capacitor_SMD:C_1206_3216Metric"
+		(property "Footprint" "Capacitor_SMD:C_0603_1608Metric"
 			(at 114.6048 72.39 0)
 			(effects
@@
 			)
 		)
-		(property "Footprint" "Capacitor_SMD:C_1206_3216Metric"
+		(property "Footprint" "Capacitor_SMD:C_0603_1608Metric"
 			(at 141.2748 39.37 0)
 			(effects

Commit message: Add datasheets, add BOM links
Signed-off-by: Mateusz Pająk <22417805+Tai-Min@users.noreply.github.com>
Parts:
- C4, C7, C8: LCSC (none) -> https://www.lcsc.com/product-detail/C66501.html
- C5: LCSC (none) -> https://www.lcsc.com/product-detail/C170142.html
- C6: value 6p / 16V -> 6p / 50V; LCSC (none) -> https://www.lcsc.com/product-detail/C170142.html
- J4: LCSC (none) -> https://www.lcsc.com/product-detail/C7494874.html; now not fitted
- J5: LCSC (none) -> https://www.lcsc.com/product-detail/C7494857.html; now not fitted
- R12: LCSC (none) -> https://www.lcsc.com/product-detail/C98220.html
- U4: LCSC (none) -> https://www.lcsc.com/product-detail/C2847904.html?s_z=n_STM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
- Y1: LCSC (none) -> https://www.lcsc.com/product-detail/C2842269.html
Changed lines of the file:
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@@
 			)
 		)
-		(property "Datasheet" "~"
+		(property "Datasheet" "\\datasheets\\HCI XC53G2-8.000-F12NJHP.pdf"
 			(at 109.22 71.12 0)
 			(effects
@@
 			)
 		)
+		(property "LCSC" "https://www.lcsc.com/product-detail/C2842269.html"
+			(at 109.22 71.12 0)
+			(effects
+				(font
+					(size 1.27 1.27)
+				)
+				(hide yes)
+			)
+		)
+		(property "Field5" ""
+			(at 109.22 71.12 0)
+			(effects
+				(font
+					(size 1.27 1.27)
+				)
+				(hide yes)
+			)
+		)
 		(pin "1"
 		)
@@
 			)
 		)
+		(property "LCSC" "https://www.lcsc.com/product-detail/C66501.html"
+			(at 91.44 73.66 90)
+			(effects
+				(font
+					(size 1.27 1.27)
+				)
+				(hide yes)
+			)
+		)
+		(property "Field5" ""
+			(at 91.44 73.66 90)
+			(effects
+				(font
+					(size 1.27 1.27)
+				)
+				(hide yes)
+			)
+		)
 		(pin "2"
 		)
@@
 		(property "Description" "Unpolarized capacitor"
 			(at 102.87 76.2 0)
+			(effects
+				(font
+					(size 1.27 1.27)
+				)
+				(hide yes)
+			)
+		)
+		(property "LCSC" "https://www.lcsc.com/product-detail/C170142.html"
+			(at 102.87 76.2 90)
+			(effects
+				(font
+					(size 1.27 1.27)
+				)
+				(hide yes)
+			)
+		)
+		(property "Field5" ""
+			(at 102.87 76.2 90)
 			(effects
 				(font
@@
 		(in_bom yes)
 		(on_board yes)
-		(dnp no)
+		(dnp yes)
 		(fields_autoplaced yes)
 		(property "Reference" "J4"
@@
 			)
 		)
+		(property "LCSC" "https://www.lcsc.com/product-detail/C7494874.html"
+			(at 100.33 106.68 0)
+			(effects
+				(font
+					(size 1.27 1.27)
+				)
+				(hide yes)
+			)
+		)
+		(property "Field5" ""
+			(at 100.33 106.68 0)
+			(effects
+				(font
+					(size 1.27 1.27)
+				)
+				(hide yes)
+			)
+		)
 		(pin "5"
 		)
@@
 			)
 		)
-		(property "Datasheet" "https://www.st.com/resource/en/datasheet/stm32g0b1cb.pdf"
+		(property "Datasheet" "\\datasheets\\stm32g0b1cb-2.pdf"
 			(at 161.29 101.6 0)
 			(effects
@@
 		)
 		(property "Description" "STMicroelectronics Arm Cortex-M0+ MCU, 128KB flash, 144KB RAM, 64 MHz, 1.7-3.6V, 44 GPIO, LQFP48"
+			(at 161.29 101.6 0)
+			(effects
+				(font
+					(size 1.27 1.27)
+				)
+				(hide yes)
+			)
+		)
+		(property "LCSC" "https://www.lcsc.com/product-detail/C2847904.html?s_z=n_STM32G0B1CBT"
+			(at 161.29 101.6 0)
+			(effects
+				(font
+					(size 1.27 1.27)
+				)
+				(hide yes)
+			)
+		)
+		(property "Field5" ""
 			(at 161.29 101.6 0)
 			(effects
@@
 			)
 		)
+		(property "LCSC" "https://www.lcsc.com/product-detail/C66501.html"
+			(at 152.4 43.18 90)
+			(effects
+				(font
+					(size 1.27 1.27)
+				)
+				(hide yes)
+			)
+		)
+		(property "Field5" ""
+			(at 152.4 43.18 90)
+			(effects
+				(font
+					(size 1.27 1.27)
+				)
+				(hide yes)
+			)
+		)
 		(pin "2"
 		)
@@
 			)
 		)
+		(property "LCSC" "https://www.lcsc.com/product-detail/C98220.html"
+			(at 99.06 134.62 0)
+			(effects
+				(font
+					(size 1.27 1.27)
+				)
+				(hide yes)
+			)
+		)
+		(property "Field5" ""
+			(at 99.06 134.62 0)
+			(effects
+				(font
+					(size 1.27 1.27)
+				)
+				(hide yes)
+			)
+		)
 		(pin "1"
 		)
@@
 		(in_bom yes)
 		(on_board yes)
-		(dnp no)
+		(dnp yes)
 		(fields_autoplaced yes)
 		(property "Reference" "J5"
@@
 			)
 		)
+		(property "LCSC" "https://www.lcsc.com/product-detail/C7494857.html"
+			(at 105.41 127 0)
+			(effects
+				(font
+					(size 1.27 1.27)
+				)
+				(hide yes)
+			)
+		)
+		(property "Field5" ""
+			(at 105.41 127 0)
+			(effects
+				(font
+					(size 1.27 1.27)
+				)
+				(hide yes)
+			)
+		)
 		(pin "2"
 		)
@@
 			)
 		)
-		(property "Value" "6p / 16V"
+		(property "Value" "6p / 50V"
 			(at 121.158 73.6601 90)
 			(effects
@@
 		(property "Description" "Unpolarized capacitor"
 			(at 115.57 76.2 0)
+			(effects
+				(font
+					(size 1.27 1.27)
+				)
+				(hide yes)
+			)
+		)
+		(property "LCSC" "https://www.lcsc.com/product-detail/C170142.html"
+			(at 115.57 76.2 90)
+			(effects
+				(font
+					(size 1.27 1.27)
+				)
+				(hide yes)
+			)
+		)
+		(property "Field5" ""
+			(at 115.57 76.2 90)
 			(effects
 				(font
@@
 			(effects
 				(font
+					(size 1.27 1.27)
+				)
+				(hide yes)
+			)
+		)
+		(property "LCSC" "https://www.lcsc.com/product-detail/C66501.html"
+			(at 142.24 43.18 90)
+			(effects
+				(font
+					(size 1.27 1.27)
+				)
+				(hide yes)
+			)
+		)
+		(property "Field5" ""
+			(at 142.24 43.18 90)
+			(effects
+				(font
