File: hw/bridge/mcu.kicad_sch (KiCad schematic)
At the start: 10 parts, among them J4 SWD, J5 BOOT, U4 STM32G0B1CBT, Y1 HCI XC53G2-8.000-F12NJHP

Commit message: Minor fixes
Signed-off-by: Mateusz Pająk <22417805+Tai-Min@users.noreply.github.com>
Parts:
- C12: renamed from C4; value 100n / 16V -> 100n
- C13: renamed from C5; value 6p / 50V -> 6p
- C14: renamed from C6; value 6p / 50V -> 6p
- C15: renamed from C7; value 100n / 16V -> 100n
- C16: renamed from C8; value 100n / 16V -> 100n
- Y2: renamed from Y1; Freq (none) -> 8MHz
- renumbered J4 to J3, J5 to J4, R12 to R11, U4 to U7
Other:
- note removed: "8MHz"
Changed lines of the file:
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@@
 	(generator_version "9.0")
 	(paper "A4")
-	(text "8MHz"
-		(exclude_from_sim no)
-		(at 109.22 75.184 0)
-		(effects
-			(font
-				(size 1.27 1.27)
-			)
-		)
-	)
 	(text "VREF/VDD"
 		(exclude_from_sim no)
@@
 		(dnp no)
 		(fields_autoplaced yes)
-		(property "Reference" "#PWR029"
+		(property "Reference" "#PWR042"
 			(at 91.44 85.09 0)
 			(effects
@@
 			(project "bridge"
 				(path "/3b0cc3d4-df75-4145-abb6-d19d57c31f1b/ee32e54e-8e22-4372-9897-0863eef95f76"
-					(reference "#PWR029")
+					(reference "#PWR042")
 					(unit 1)
 				)
@@
 		(dnp no)
 		(fields_autoplaced yes)
-		(property "Reference" "#PWR034"
+		(property "Reference" "#PWR047"
 			(at 132.08 63.5 0)
 			(effects
@@
 			(project "bridge"
 				(path "/3b0cc3d4-df75-4145-abb6-d19d57c31f1b/ee32e54e-8e22-4372-9897-0863eef95f76"
-					(reference "#PWR034")
+					(reference "#PWR047")
 					(unit 1)
 				)
@@
 		(on_board yes)
 		(dnp no)
-		(property "Reference" "Y1"
+		(property "Reference" "Y2"
 			(at 108.966 67.056 0)
 			(effects
@@
 			)
 		)
-		(property "Field5" ""
-			(at 109.22 71.12 0)
-			(effects
-				(font
-					(size 1.27 1.27)
-				)
-				(hide yes)
+		(property "Freq" "8MHz"
+			(at 109.22 75.184 0)
+			(effects
+				(font
+					(size 1.27 1.27)
+				)
 			)
 		)
@@
 			(project ""
 				(path "/3b0cc3d4-df75-4145-abb6-d19d57c31f1b/ee32e54e-8e22-4372-9897-0863eef95f76"
-					(reference "Y1")
+					(reference "Y2")
 					(unit 1)
 				)
@@
 		(on_board yes)
 		(dnp no)
-		(property "Reference" "C4"
+		(property "Reference" "C12"
 			(at 85.598 72.898 90)
 			(effects
@@
 			)
 		)
-		(property "Value" "100n / 16V"
+		(property "Value" "100n"
 			(at 87.63 71.6281 90)
 			(effects
@@
 			(project "bridge"
 				(path "/3b0cc3d4-df75-4145-abb6-d19d57c31f1b/ee32e54e-8e22-4372-9897-0863eef95f76"
-					(reference "C4")
+					(reference "C12")
 					(unit 1)
 				)
@@
 		(on_board yes)
 		(dnp no)
-		(property "Reference" "C5"
+		(property "Reference" "C13"
 			(at 97.028 75.438 90)
 			(effects
@@
 			)
 		)
-		(property "Value" "6p / 50V"
-			(at 99.06 74.1681 90)
+		(property "Value" "6p"
+			(at 99.06 75.692 90)
 			(effects
 				(font
@@
 			(project "bridge"
 				(path "/3b0cc3d4-df75-4145-abb6-d19d57c31f1b/ee32e54e-8e22-4372-9897-0863eef95f76"
-					(reference "C5")
+					(reference "C13")
 					(unit 1)
 				)
@@
 		(on_board yes)
 		(dnp no)
-		(property "Reference" "#PWR038"
+		(property "Reference" "#PWR051"
 			(at 152.4 54.61 0)
 			(effects
@@
 			(project "bridge"
 				(path "/3b0cc3d4-df75-4145-abb6-d19d57c31f1b/ee32e54e-8e22-4372-9897-0863eef95f76"
-					(reference "#PWR038")
+					(reference "#PWR051")
 					(unit 1)
 				)
@@
 		(dnp no)
 		(fields_autoplaced yes)
-		(property "Reference" "#PWR033"
+		(property "Reference" "#PWR046"
 			(at 109.22 88.9 0)
 			(effects
@@
 			(project "bridge"
 				(path "/3b0cc3d4-df75-4145-abb6-d19d57c31f1b/ee32e54e-8e22-4372-9897-0863eef95f76"
-					(reference "#PWR033")
+					(reference "#PWR046")
 					(unit 1)
 				)
@@
 		(on_board yes)
 		(dnp no)
-		(property "Reference" "#PWR036"
+		(property "Reference" "#PWR049"
 			(at 142.24 54.61 0)
 			(effects
@@
 			(project "bridge"
 				(path "/3b0cc3d4-df75-4145-abb6-d19d57c31f1b/ee32e54e-8e22-4372-9897-0863eef95f76"
-					(reference "#PWR036")
+					(reference "#PWR049")
 					(unit 1)
 				)
@@
 		(dnp yes)
 		(fields_autoplaced yes)
-		(property "Reference" "J4"
+		(property "Reference" "J3"
 			(at 101.6 97.79 0)
 			(effects
@@
 			(project ""
 				(path "/3b0cc3d4-df75-4145-abb6-d19d57c31f1b/ee32e54e-8e22-4372-9897-0863eef95f76"
-					(reference "J4")
+					(reference "J3")
 					(unit 1)
 				)
@@
 		(dnp no)
 		(fields_autoplaced yes)
-		(property "Reference" "#PWR031"
+		(property "Reference" "#PWR044"
 			(at 99.06 129.54 0)
 			(effects
@@
 			(project "bridge"
 				(path "/3b0cc3d4-df75-4145-abb6-d19d57c31f1b/ee32e54e-8e22-4372-9897-0863eef95f76"
-					(reference "#PWR031")
+					(reference "#PWR044")
 					(unit 1)
 				)
@@
 		(on_board yes)
 		(dnp no)
-		(property "Reference" "U4"
+		(property "Reference" "U7"
 			(at 164.592 149.352 0)
 			(effects
@@
 			(project "bridge"
 				(path "/3b0cc3d4-df75-4145-abb6-d19d57c31f1b/ee32e54e-8e22-4372-9897-0863eef95f76"
-					(reference "U4")
+					(reference "U7")
 					(unit 1)
 				)
@@
 		(dnp no)
 		(fields_autoplaced yes)
-		(property "Reference" "#PWR035"
+		(property "Reference" "#PWR048"
 			(at 142.24 41.91 0)
 			(effects
@@
 			(project "bridge"
 				(path "/3b0cc3d4-df75-4145-abb6-d19d57c31f1b/ee32e54e-8e22-4372-9897-0863eef95f76"
-					(reference "#PWR035")
+					(reference "#PWR048")
 					(unit 1)
 				)
@@
 		(on_board yes)
 		(dnp no)
-		(property "Reference" "C8"
+		(property "Reference" "C16"
 			(at 146.558 42.418 90)
 			(effects
@@
 			)
 		)
-		(property "Value" "100n / 16V"
+		(property "Value" "100n"
 			(at 148.59 41.1481 90)
 			(effects
@@
 			(project "bridge"
 				(path "/3b0cc3d4-df75-4145-abb6-d19d57c31f1b/ee32e54e-8e22-4372-9897-0863eef95f76"
-					(reference "C8")
+					(reference "C16")
 					(unit 1)
 				)
@@
 		(dnp no)
 		(fields_autoplaced yes)
-		(property "Reference" "#PWR028"
+		(property "Reference" "#PWR041"
 			(at 83.82 114.3 0)
 			(effects
@@
 			(project ""
 				(path "/3b0cc3d4-df75-4145-abb6-d19d57c31f1b/ee32e54e-8e22-4372-9897-0863eef95f76"
-					(reference "#PWR028")
+					(reference "#PWR041")
 					(unit 1)
 				)
@@
 		(dnp no)
 		(fields_autoplaced yes)
-		(property "Reference" "#PWR040"
+		(property "Reference" "#PWR053"
 			(at 162.56 54.61 0)
 			(effects
@@
 			(project "bridge"
 				(path "/3b0cc3d4-df75-4145-abb6-d19d57c31f1b/ee32e54e-8e22-4372-9897-0863eef95f76"
-					(reference "#PWR040")
+					(reference "#PWR053")
 					(unit 1)
 				)
@@
 		(dnp no)
 		(fields_autoplaced yes)
-		(property "Reference" "#PWR037"
+		(property "Reference" "#PWR050"
 			(at 152.4 41.91 0)
 			(effects
@@
 			(project "bridge"
 				(path "/3b0cc3d4-df75-4145-abb6-d19d57c31f1b/ee32e54e-8e22-4372-9897-0863eef95f76"
-					(reference "#PWR037")
+					(reference "#PWR050")
 					(unit 1)
 				)
@@
 		(dnp no)
 		(fields_autoplaced yes)
-		(property "Reference" "#PWR039"
+		(property "Reference" "#PWR052"
 			(at 161.29 157.48 0)
 			(effects
@@
 			(project "bridge"
 				(path "/3b0cc3d4-df75-4145-abb6-d19d57c31f1b/ee32e54e-8e22-4372-9897-0863eef95f76"
-					(reference "#PWR039")
+					(reference "#PWR052")
 					(unit 1)
 				)
@@
 		(dnp no)
 		(fields_autoplaced yes)
-		(property "Reference" "R12"
+		(property "Reference" "R11"
 			(at 101.6 133.3499 0)
 			(effects
@@
 			(project ""
 				(path "/3b0cc3d4-df75-4145-abb6-d19d57c31f1b/ee32e54e-8e22-4372-9897-0863eef95f76"
-					(reference "R12")
+					(reference "R11")
 					(unit 1)
 				)
@@
 		(dnp yes)
 		(fields_autoplaced yes)
-		(property "Reference" "J5"
+		(property "Reference" "J4"
 			(at 107.95 126.9999 0)
 			(effects
@@
 			(project ""
 				(path "/3b0cc3d4-df75-4145-abb6-d19d57c31f1b/ee32e54e-8e22-4372-9897-0863eef95f76"
-					(reference "J5")
+					(reference "J4")
 					(unit 1)
 				)
@@
 		(on_board yes)
 		(dnp no)
-		(property "Reference" "C6"
+		(property "Reference" "C14"
 			(at 119.126 74.93 90)
 			(effects
@@
 			)
 		)
-		(property "Value" "6p / 50V"
-			(at 121.158 73.6601 90)
+		(property "Value" "6p"
+			(at 121.158 75.184 90)
 			(effects
 				(font
@@
 			(project "bridge"
 				(path "/3b0cc3d4-df75-4145-abb6-d19d57c31f1b/ee32e54e-8e22-4372-9897-0863eef95f76"
-					(reference "C6")
+					(reference "C14")
 					(unit 1)
 				)
@@
 		(dnp no)
 		(fields_autoplaced yes)
-		(property "Reference" "#PWR030"
+		(property "Reference" "#PWR043"
 			(at 92.71 105.41 0)
 			(effects
@@
 			(project ""
 				(path "/3b0cc3d4-df75-4145-abb6-d19d57c31f1b/ee32e54e-8e22-4372-9897-0863eef95f76"
-					(reference "#PWR030")
+					(reference "#PWR043")
 					(unit 1)
 				)
@@
 		(on_board yes)
 		(dnp no)
-		(property "Reference" "C7"
+		(property "Reference" "C15"
 			(at 136.398 42.418 90)
 			(effects
@@
 			)
 		)
-		(property "Value" "100n / 16V"
+		(property "Value" "100n"
 			(at 138.43 41.1481 90)
 			(effects
@@
 			(project "bridge"
 				(path "/3b0cc3d4-df75-4145-abb6-d19d57c31f1b/ee32e54e-8e22-4372-9897-0863eef95f76"
-					(reference "C7")
+					(reference "C15")
 					(unit 1)
 				)
@@
 		(dnp no)
 		(fields_autoplaced yes)
-		(property "Reference" "#PWR032"
+		(property "Reference" "#PWR045"
 			(at 99.06 146.05 0)
 			(effects
@@
 			(project "bridge"
 				(path "/3b0cc3d4-df75-4145-abb6-d19d57c31f1b/ee32e54e-8e22-4372-9897-0863eef95f76"
-					(reference "#PWR032")
+					(reference "#PWR045")
 					(unit 1)
 				)

Commit message: Fix annotation error
Signed-off-by: Mateusz Pająk <22417805+Tai-Min@users.noreply.github.com>
Parts:
- renumbered C12 to C11, C13 to C12, C14 to C13, C15 to C14, C16 to C15, R11 to R16
Changed lines of the file:
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@@
 		(on_board yes)
 		(dnp no)
-		(property "Reference" "C12"
+		(property "Reference" "C11"
 			(at 85.598 72.898 90)
 			(effects
@@
 			(project "bridge"
 				(path "/3b0cc3d4-df75-4145-abb6-d19d57c31f1b/ee32e54e-8e22-4372-9897-0863eef95f76"
-					(reference "C12")
+					(reference "C11")
 					(unit 1)
 				)
@@
 		(on_board yes)
 		(dnp no)
-		(property "Reference" "C13"
+		(property "Reference" "C12"
 			(at 97.028 75.438 90)
 			(effects
@@
 			(project "bridge"
 				(path "/3b0cc3d4-df75-4145-abb6-d19d57c31f1b/ee32e54e-8e22-4372-9897-0863eef95f76"
-					(reference "C13")
+					(reference "C12")
 					(unit 1)
 				)
@@
 		(on_board yes)
 		(dnp no)
-		(property "Reference" "C16"
+		(property "Reference" "C15"
 			(at 146.558 42.418 90)
 			(effects
@@
 			(project "bridge"
 				(path "/3b0cc3d4-df75-4145-abb6-d19d57c31f1b/ee32e54e-8e22-4372-9897-0863eef95f76"
-					(reference "C16")
+					(reference "C15")
 					(unit 1)
 				)
@@
 		(dnp no)
 		(fields_autoplaced yes)
-		(property "Reference" "R11"
+		(property "Reference" "R16"
 			(at 101.6 133.3499 0)
 			(effects
@@
 			(project ""
 				(path "/3b0cc3d4-df75-4145-abb6-d19d57c31f1b/ee32e54e-8e22-4372-9897-0863eef95f76"
-					(reference "R11")
+					(reference "R16")
 					(unit 1)
 				)
@@
 		(on_board yes)
 		(dnp no)
-		(property "Reference" "C14"
+		(property "Reference" "C13"
 			(at 119.126 74.93 90)
 			(effects
@@
 			(project "bridge"
 				(path "/3b0cc3d4-df75-4145-abb6-d19d57c31f1b/ee32e54e-8e22-4372-9897-0863eef95f76"
-					(reference "C14")
+					(reference "C13")
 					(unit 1)
 				)
@@
 		(on_board yes)
 		(dnp no)
-		(property "Reference" "C15"
+		(property "Reference" "C14"
 			(at 136.398 42.418 90)
 			(effects
@@
 			(project "bridge"
 				(path "/3b0cc3d4-df75-4145-abb6-d19d57c31f1b/ee32e54e-8e22-4372-9897-0863eef95f76"
-					(reference "C15")
-					(unit 1)
-				)
+					(reference "C14")
+					(unit 1)
+				)

Commit message: Manufacture fixes
Signed-off-by: Mateusz Pająk <22417805+Tai-Min@users.noreply.github.com>
Parts:
- R16: value 10k -> 10K
Changed lines of the file:
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@@
 			)
 		)
-		(property "Value" "10k"
+		(property "Value" "10K"
 			(at 101.6 135.8899 0)
 			(effects
