File: hw/mcu/mcu.kicad_pcb (KiCad board)
At the start: 2 copper layers, 0 parts

Commit message: Add board2pdf
Signed-off-by: Mateusz Pająk <22417805+Tai-Min@users.noreply.github.com>
Parts:
- added REF**: Smolhaj_Scale_0.1, Symbol:Smolhaj_Scale_0.1, F.Cu at (180.7, 77.3)
Other:
- board outline added: 64.1 x 33.7 mm
