File: hw/bus_connector/bus_connector.kicad_pcb (KiCad board)
At the start: 2 copper layers, 70 x 36 mm, 18 parts, among them J1 DE9_Left, J2 DE9_Top, J3 DE9_Right

Commit message: Minor changes
Signed-off-by: Mateusz Pająk <22417805+Tai-Min@users.noreply.github.com>
Routing:
- net GND: vias 454 -> 464
Changed lines of the file:
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@@
 	)
 	(via
+		(at 126.49 113.55)
+		(size 0.45)
+		(drill 0.3)
+		(layers "F.Cu" "B.Cu")
+		(free yes)
+		(net 2)
+	)
+	(via
 		(at 112.5 105.5)
 		(size 0.45)
@@
 	)
 	(via
+		(at 174.74 103.69)
+		(size 0.45)
+		(drill 0.3)
+		(layers "F.Cu" "B.Cu")
+		(free yes)
+		(net 2)
+	)
+	(via
 		(at 147.5 89.5)
 		(size 0.45)
@@
 	)
 	(via
+		(at 173.74 108.47)
+		(size 0.45)
+		(drill 0.3)
+		(layers "F.Cu" "B.Cu")
+		(free yes)
+		(net 2)
+	)
+	(via
 		(at 156.5 116.095)
 		(size 0.45)
@@
 	)
 	(via
+		(at 173.7 111.31)
+		(size 0.45)
+		(drill 0.3)
+		(layers "F.Cu" "B.Cu")
+		(free yes)
+		(net 2)
+	)
+	(via
 		(at 150.5 111.015)
 		(size 0.45)
@@
 	)
 	(via
+		(at 126.49 121.17)
+		(size 0.45)
+		(drill 0.3)
+		(layers "F.Cu" "B.Cu")
+		(free yes)
+		(net 2)
+	)
+	(via
 		(at 124.5 105.935)
 		(size 0.45)
@@
 	)
 	(via
+		(at 168.66 99.56)
+		(size 0.45)
+		(drill 0.3)
+		(layers "F.Cu" "B.Cu")
+		(free yes)
+		(net 2)
+	)
+	(via
 		(at 128.55 97.825)
 		(size 0.45)
@@
 	)
 	(via
+		(at 128.33 106.86)
+		(size 0.45)
+		(drill 0.3)
+		(layers "F.Cu" "B.Cu")
+		(free yes)
+		(net 2)
+	)
+	(via
 		(at 155.5 93)
 		(size 0.45)
@@
 	)
 	(via
-		(at 126.5 98.315)
+		(at 126.35 97.84)
 		(size 0.45)
 		(drill 0.3)
@@
 	)
 	(via
+		(at 126.49 116.09)
+		(size 0.45)
+		(drill 0.3)
+		(layers "F.Cu" "B.Cu")
+		(free yes)
+		(net 2)
+	)
+	(via
 		(at 112.5 123.5)
 		(size 0.45)
@@
 	)
 	(via
+		(at 126.49 118.63)
+		(size 0.45)
+		(drill 0.3)
+		(layers "F.Cu" "B.Cu")
+		(free yes)
+		(net 2)
+	)
+	(via
 		(at 114.5 108.475)
 		(size 0.45)
@@
 	)
 	(via
+		(at 164.84 96.9)
+		(size 0.45)
+		(drill 0.3)
+		(layers "F.Cu" "B.Cu")
+		(free yes)
+		(net 2)
+	)
+	(via
 		(at 139.5 89.5)
 		(size 0.45)
@@
 	)
 	(segment
-		(start 127.3 102.5125)
+		(start 134.170086 103.48)
 		(end 128.2675 103.48)
 		(width 0.2)
@@
 	)
 	(segment
-		(start 124.472291 102.5125)
-		(end 124.363351 102.5125)
-		(width 0.2)
-		(layer "F.Cu")
-		(net 7)
-	)
-	(segment
-		(start 134.820624 102.82946)
-		(end 135.033188 102.616898)
+		(start 148.706788 104.735)
+		(end 148.264914 104.735)
 		(width 0.2)
 		(layer "F.Cu")
@@
 	)
 	(segment
-		(start 132.317066 103.279122)
-		(end 132.526188 103.279122)
+		(start 124.472291 102.5125)
+		(end 124.363351 102.5125)
 		(width 0.2)
 		(layer "F.Cu")
@@
 	)
 	(segment
-		(start 136.215086 101.435)
-		(end 144.964914 101.435)
-		(width 0.2)
-		(layer "F.Cu")
-		(net 7)
-	)
-	(segment
 		(start 123.68 104.525)
 		(end 122.5 105.705)
@@
 	)
 	(segment
-		(start 150.55 104.35)
-		(end 150.55 104.25)
-		(width 0.2)
-		(layer "F.Cu")
-		(net 7)
-	)
-	(segment
-		(start 132.936188 103.48)
-		(end 134.170086 103.48)
-		(width 0.2)
-		(layer "F.Cu")
-		(net 7)
-	)
-	(segment
 		(start 125.288602 102.793999)
 		(end 125.1601 102.793999)
@@
 	)
 	(segment
-		(start 128.2675 103.48)
-		(end 132.116188 103.48)
+		(start 157.692644 106.318844)
+		(end 157.774644 106.318844)
 		(width 0.2)
 		(layer "F.Cu")
@@
 	)
 	(segment
-		(start 157.692644 106.318844)
-		(end 157.774644 106.318844)
+		(start 147.72681 104.196896)
+		(end 144.964914 101.435)
 		(width 0.2)
 		(layer "F.Cu")
@@
 	(segment
 		(start 148.264914 104.735)
-		(end 150.165 104.735)
-		(width 0.2)
-		(layer "F.Cu")
-		(net 7)
-	)
-	(segment
-		(start 144.964914 101.435)
-		(end 148.264914 104.735)
+		(end 147.72681 104.196896)
 		(width 0.2)
 		(layer "F.Cu")
@@
 	)
 	(segment
-		(start 150.165 104.735)
-		(end 150.55 104.35)
-		(width 0.2)
-		(layer "F.Cu")
-		(net 7)
-	)
-	(segment
 		(start 125.429351 102.5125)
 		(end 125.429351 102.65325)
@@
 	)
 	(segment
-		(start 135.033188 102.616898)
-		(end 136.215086 101.435)
+		(start 128.2675 103.48)
+		(end 127.3 102.5125)
 		(width 0.2)
 		(layer "F.Cu")
@@
 	)
 	(segment
-		(start 132.727066 103.48)
-		(end 132.936188 103.48)
-		(width 0.2)
-		(layer "F.Cu")
-		(net 7)
-	)
-	(segment
 		(start 159.578644 106.482852)
 		(end 159.578644 106.516)
@@
 	)
 	(segment
-		(start 134.170086 103.48)
-		(end 134.820624 102.82946)
-		(width 0.2)
-		(layer "F.Cu")
-		(net 7)
-	)
-	(segment
 		(start 157.938644 106.482844)
 		(end 157.938644 106.516)
@@
 	)
 	(segment
+		(start 150.55 104.25)
+		(end 150.55 104.35)
+		(width 0.2)
+		(layer "F.Cu")
+		(net 7)
+	)
+	(segment
 		(start 157.528644 106.516)
 		(end 157.528644 106.482844)
@@
 	)
 	(segment
+		(start 148.915852 104.735)
+		(end 148.706788 104.735)
+		(width 0.2)
+		(layer "F.Cu")
+		(net 7)
+	)
+	(segment
 		(start 127.3 102.5125)
 		(end 126.003351 102.5125)
@@
 	)
 	(segment
+		(start 136.215086 101.435)
+		(end 134.170086 103.48)
+		(width 0.2)
+		(layer "F.Cu")
+		(net 7)
+	)
+	(segment
+		(start 150.55 104.35)
+		(end 150.165 104.735)
+		(width 0.2)
+		(layer "F.Cu")
+		(net 7)
+	)
+	(segment
 		(start 156.943858 106.68)
 		(end 157.364644 106.68)
@@
 		(net 7)
 	)
+	(segment
+		(start 150.165 104.735)
+		(end 149.526788 104.735)
+		(width 0.2)
+		(layer "F.Cu")
+		(net 7)
+	)
+	(segment
+		(start 144.964914 101.435)
+		(end 136.215086 101.435)
+		(width 0.2)
+		(layer "F.Cu")
+		(net 7)
+	)
+	(segment
+		(start 149.325852 104.534064)
+		(end 149.116788 104.534064)
+		(width 0.2)
+		(layer "F.Cu")
+		(net 7)
+	)
 	(via
 		(at 150.55 104.25)
@@
 	)
 	(arc
-		(start 132.116188 103.48)
-		(mid 132.187209 103.450582)
-		(end 132.216627 103.379561)
-		(width 0.2)
-		(layer "F.Cu")
-		(net 7)
-	)
-	(arc
 		(start 157.364644 106.68)
 		(mid 157.48061 106.631966)
@@
 	)
 	(arc
-		(start 132.526188 103.279122)
-		(mid 132.597209 103.30854)
-		(end 132.626627 103.379561)
-		(width 0.2)
-		(layer "F.Cu")
-		(net 7)
-	)
-	(arc
 		(start 124.746411 102.23838)
 		(mid 124.649495 102.278524)
@@
 	)
 	(arc
-		(start 132.216627 103.379561)
-		(mid 132.246045 103.30854)
-		(end 132.317066 103.279122)
+		(start 149.01632 104.634532)
+		(mid 148.986894 104.705574)
+		(end 148.915852 104.735)
+		(width 0.2)
+		(layer "F.Cu")
+		(net 7)
+	)
+	(arc
+		(start 149.116788 104.534064)
+		(mid 149.045746 104.56349)
+		(end 149.01632 104.634532)
 		(width 0.2)
 		(layer "F.Cu")
@@
 	)
 	(arc
+		(start 149.42632 104.634532)
+		(mid 149.396894 104.56349)
+		(end 149.325852 104.534064)
+		(width 0.2)
+		(layer "F.Cu")
+		(net 7)
+	)
+	(arc
 		(start 157.938644 106.516)
 		(mid 157.986678 106.631966)
@@
 	)
 	(arc
-		(start 132.626627 103.379561)
-		(mid 132.656045 103.450582)
-		(end 132.727066 103.48)
+		(start 149.526788 104.735)
+		(mid 149.455746 104.705574)
+		(end 149.42632 104.634532)
 		(width 0.2)
 		(layer "F.Cu")
@@
 		(base_line
 			(pts
-				(xy 132.116188 103.48) (xy 134.170086 103.48) (xy 135.033188 102.616898)
+				(xy 149.526788 104.735) (xy 148.264914 104.735) (xy 147.72681 104.196896)
 			)
 		)
 		(base_line_coupled
 			(pts
-				(xy 132.116188 103.89) (xy 132.138184 103.89)
+				(xy 149.593394 104.735) (xy 149.582391 104.735)
 			)
 		)
 		(corner_radius_percent 80)
 		(end
-			(xy 135.033188 102.616898)
+			(xy 147.72681 104.196896)
 		)
-		(initial_side "left")
+		(initial_side "right")
 		(last_diff_pair_gap 0.18)
 		(last_netname "/MODBUS-")
 		(last_status "tuned")
 		(last_track_width 0.2)
-		(last_tuning "-0.0000 mm (tuned)")
+		(last_tuning "-0.0001 mm (tuned)")
 		(max_amplitude 0.4)
 		(min_amplitude 0.2)
 		(min_spacing 0.25)
 		(origin
-			(xy 132.116188 103.48)
+			(xy 149.526788 104.735)
 		)
 		(override_custom_rules no)
@@
 		(target_skew_min -0.1)
 		(tuning_mode "diff_pair_skew")
-		(members "052f6c0d-d4bf-41e4-9c5d-874dd853f8e6" "19dee752-2155-49fd-97f5-b14e5f23135b"
-			"22464d10-b8be-4f47-8e55-e0e8d38392ff" "44b2982d-6436-417f-93d5-af3c4a722c15"
-			"60a27522-3d92-4b6c-ad6d-be67ca83e1e5" "688608e6-9e72-4087-88a5-2e835f3660a3"
-			"8def1bc1-228a-410f-b339-2df6c9defc57" "9eeb910e-a2e1-4ada-9c9f-86cf219bfc6d"
-			"f967bb3c-8ac2-49e0-a588-b6d5befdacf6"
+		(members "1687dca5-8f20-4e22-9039-4569701c7e40" "626ef436-c85a-4d2c-9f9a-563af69c1a2a"
+			"67f2a8a5-ef6c-4091-b41f-98d358cf0300" "6aec65fd-2417-40a3-a25b-7f80a648e9ab"
+			"a14b04be-9ec9-42cd-b056-b9c74710d567" "cb831ba0-09c0-4659-ad54-6492e0676fb4"
+			"e4891902-01b8-43eb-9f4c-f1a274f41ecf" "fdae6fdb-0d76-4762-8423-77f1b7ac66e9"
 		)
 	)

Commit message: Add proper drawing sheet with license
Signed-off-by: Mateusz Pająk <22417805+Tai-Min@users.noreply.github.com>
Other:
- board text removed: "This documentation describes Open Hardware and is licensed under the CERN OHL v. 1.2. You may redistribute and modify this documentation under the terms of the CERN OHL v.1.2.(http://ohwr.org/cernohl). This documentation is distributed WITHOUT ANY EXPRESS OR IMPLIED WARRANTY, INCLUDING OF MERCHANTABILITY, SATISFACTORY QUALITY AND FITNESS FOR A PARTICULAR PURPOSE. Please see the CERN OHL v.1.2 for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"
Changed lines of the file:
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@@
 		)
 	)
-	(gr_text "This documentation describes Open Hardware and is licensed under the CERN OHL v. 1.2.\nYou may redistribute and modify this documentation under the terms of the CERN OHL v.1.2.(http://ohwr.org/cernohl).\nThis documentation is distributed WITHOUT ANY EXPRESS OR IMPLIED WARRANTY, INCLUDING OF MERCHANTABILITY,\nSATISFACTORY QUALITY AND FITNESS FOR A PARTICULAR PURPOSE. Please see the CERN OHL v.1.2 for applicable conditions"
-		(at 184.29 176.58 0)
-		(layer "User.4")
-		(effects
-			(font
-				(size 1 1)
-				(thickness 0.2)
-				(bold yes)
-			)
-			(justify left bottom)
-		)
-	)
 	(dimension
 		(type orthogonal)
@@
 	)
 	(embedded_fonts no)
+	(embedded_files
+		(file
+			(name "drawing_sheet.kicad_wks")
+			(type worksheet)
+			(data |KLUv/WAhCq0bANZtjiDgWjeUd7GfIpdQ3hsyJE4imh40WCrg3bHZNmcww0sw4IEAhQCDAL5lJzOj
+				pT+67/YvbT+xKmvrmW/8KFQ2Oef8xK9I+Farb213mmX+KIu3+RqV985lKu8S6eqtOr4kbVGiPXrU
+				0FVt89I+L+vxRQ2dVv1fN92t3wUAICBIqfanm+bIRNk9X4SmMtd5W/34SYZGrTXBbZzjfFP9qwIg
+				IEhPLNFpzXsqBJlvi9J55PpTNhS/0Av/dccTzaUrOLDziasXG43MLVVTuGOrGQ04il9HJPEioAVG
+				6LTOt1od2sIZjdhHehLRxxlHEEbwx28r0Vq79G/8prtGd6cqU8d59Vxc51tZlltNFAAb51H1jvM0
+				p7Ka+W79Lne3JTrOt87V0ia+237qtX6ss7lR3wKlAg6Nsqco/XufGbVV5dU7vedrd1mUqzIIhzRO
+				q66t/FLReEb8Iv6l7fpPrPLzU/zmRT29fmLrry3r1Lbi+FMaT7+82kz/dJzvtiozn57eErfgOgej
+				Qnoh+X2VsdFIaAqMl/ku4OROzIvafZ2hbfW7kCCJ7ktylavn9f1fGgeI2OAEAwGBgds6bcG5o+HQ
+				GOk9cTb90dKaF02lrP+n/ql9NMQh7Rs1ocgJXfQunAhIil7o3iRDghOXeJyNg0QNGfEmI0h6Iw6B
+				FxDiVSLih/GJxikZUMK5RDKgH0BkxhNFz+OSD7yEGNBFjY/jJ4afz0EZz0mOpkKCntM1A1rKWL+J
+				IOmsaVYpIxCP1N4BgIagATmGmBkakSCSpCDJcGBExMxVN+ZEMIr2+Ixg+w44oI2QkWfDYQBGWKkF
+				Mwg4uwAUEVRASQ6CoSO7wOH2oRcJQ92PVxKzOyKxApiF5j1bCYde/8e8NSfJCOTZBjnL5kEgk9zl
+				MlBII26C1dPzpy84m5fIib7lme/qD5PyoQz2EJoQE1jDRgTxITi8ia/sl5+zrDxPhKBBn57ycYJg
+				ZCwqHFwyZdBoqHYp0zBZO06dzgfsT4kYixZyxQyfvGf1jGnpkx8aKmozkcOWchtBzaWzZv2hQIju
+				lOqJaiUvzvCA3LzBdbUVIJOYJSx0+3ufDFvX5dIvDoxARYL0gCYirRADAnCnk8CcCCxLwcP0pwGD
+				AcdTPbjcedGBdAsSMjEiw0/8xNymVps2TR/W8jcsl1Bj2egAHQNMBQ==|
+			)
+			(checksum "F4CA3C5331BFF1A6D590C818164A77B8")
+		)
+	)
 )
