File: hw/shield/shield.kicad_pcb (KiCad board)
At the start: 2 copper layers, 31.2 x 64.5 mm, 4 parts, among them J2 DE9, U2 MAX485E, U3 TPS5405DR

Commit message: WIP shield
Signed-off-by: Mateusz Pająk <22417805+Tai-Min@users.noreply.github.com>
Parts:
- added D1: CDSOT23-T24CAN, Package_TO_SOT_SMD:SOT-23, F.Cu at (214.7, 84.7)
- added D2: SM712-02HTG, Package_TO_SOT_SMD:SOT-23, F.Cu at (214.7, 89.3)
- added RN1: 10K, Resistor_THT:R_Array_SIP9, F.Cu at (214.3, 80.2)
- added SW1: SW_DIP_x08, Button_Switch_SMD:SW_DIP_SPSTx08_Slide_KingTek_DSHP08TS_W7.62mm_P1.27mm, F.Cu at (152.6, 96.5)
- added TP1: TestPoint, TestPoint:TestPoint_Pad_D1.5mm, F.Cu at (181.8, 81.4)
- added TP2: TestPoint, TestPoint:TestPoint_Pad_D1.5mm, F.Cu at (181.8, 84.9)
- added TP3: TestPoint, TestPoint:TestPoint_Pad_D1.5mm, F.Cu at (181.8, 88.5)
- added TP4: TestPoint, TestPoint:TestPoint_Pad_D1.5mm, F.Cu at (181.8, 92.0)
- added U1: TCAN330G, Package_SO:SOIC-8-1EP_3.9x4.9mm_P1.27mm_EP2.29x3mm, F.Cu at (198.2, 94.6)
- added U4: 74HC165, Package_SO:SOIC-16_3.9x9.9mm_P1.27mm, F.Cu at (198.2, 85.5)
- moved U3 78.5 mm to (230.3, 103.9)
- moved U2 77.6 mm to (230.1, 90.2)
Connections:
- A2 pad 36: unconnected-(A2-3V3-Pad36) -> +3.3V
- A2 pad 39: unconnected-(A2-VSYS-Pad39) -> Net-(A2-VSYS)
- A2 pad 40: unconnected-(A2-VBUS-Pad40) -> Net-(A2-VBUS)
- U2 pad 1: unconnected-(U2-RO-Pad1) -> /RS_RO
- U2 pad 2: unconnected-(U2-~{RE}-Pad2) -> /RS_TNOW
- U2 pad 3: unconnected-(U2-DE-Pad3) -> /RS_TNOW
- U2 pad 4: unconnected-(U2-DI-Pad4) -> /RS_DI
- U2 pad 5: unconnected-(U2-GND-Pad5) -> GND
- U2 pad 6: unconnected-(U2-A-Pad6) -> Net-(U2-A)
- U2 pad 7: unconnected-(U2-B-Pad7) -> Net-(U2-B)
- U2 pad 8: unconnected-(U2-VCC-Pad8) -> +3.3V
- U3 pad 1: unconnected-(U3-BOOT-Pad1) -> Net-(U3-BOOT)
- U3 pad 2: unconnected-(U3-VIN-Pad2) -> Net-(D4-K)
- U3 pad 3: unconnected-(U3-ROSC-Pad3) -> Net-(U3-ROSC)
- U3 pad 4: unconnected-(U3-SS-Pad4) -> Net-(U3-SS)
- U3 pad 5: unconnected-(U3-VSENSE-Pad5) -> +5V
- U3 pad 6: unconnected-(U3-COMP-Pad6) -> Net-(U3-COMP)
- U3 pad 7: unconnected-(U3-GND-Pad7) -> GND
- U3 pad 8: unconnected-(U3-LX-Pad8) -> Net-(D3-K)
Other:
- board text removed: "This documentation describes Open Hardware and is licensed under the CERN OHL v. 1.2. You may redistribute and modify this documentation under the terms of the CERN OHL v.1.2.(http://ohwr.org/cernohl). This documentation is distributed WITHOUT ANY EXPRESS OR IMPLIED WARRANTY, INCLUDING OF MERCHANTABILITY, SATISFACTORY QUALITY AND FITNESS FOR A PARTICULAR PURPOSE. Please see the CERN OHL v.1.2 for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"
