File: hw/shield/shield.kicad_pcb (KiCad board)
At the start: 2 copper layers, 31.2 x 64.5 mm, 4 parts, among them J2 DE9, U2 MAX485E, U3 TPS5405DR

Commit message: WIP shield
Signed-off-by: Mateusz Pająk <22417805+Tai-Min@users.noreply.github.com>
Parts:
- added D1: CDSOT23-T24CAN, Package_TO_SOT_SMD:SOT-23, F.Cu at (214.7, 84.7)
- added D2: SM712-02HTG, Package_TO_SOT_SMD:SOT-23, F.Cu at (214.7, 89.3)
- added RN1: 10K, Resistor_THT:R_Array_SIP9, F.Cu at (214.3, 80.2)
- moved U3 78.5 mm to (230.3, 103.9)
- moved U2 77.6 mm to (230.1, 90.2)
Connections:
- A2 pad 36: unconnected-(A2-3V3-Pad36) -> +3.3V
- U2 pad 1: unconnected-(U2-RO-Pad1) -> /RO
- U2 pad 2: unconnected-(U2-~{RE}-Pad2) -> /TNOW
- U2 pad 3: unconnected-(U2-DE-Pad3) -> /TNOW
- U2 pad 4: unconnected-(U2-DI-Pad4) -> /DI
- U2 pad 5: unconnected-(U2-GND-Pad5) -> GND
- U2 pad 6: unconnected-(U2-A-Pad6) -> Net-(U2-A)
- U2 pad 7: unconnected-(U2-B-Pad7) -> Net-(U2-B)
- U2 pad 8: unconnected-(U2-VCC-Pad8) -> +3.3V
Other:
- board text removed: "This documentation describes Open Hardware and is licensed under the CERN OHL v. 1.2. You may redistribute and modify this documentation under the terms of the CERN OHL v.1.2.(http://ohwr.org/cernohl). This documentation is distributed WITHOUT ANY EXPRESS OR IMPLIED WARRANTY, INCLUDING OF MERCHANTABILITY, SATISFACTORY QUALITY AND FITNESS FOR A PARTICULAR PURPOSE. Please see the CERN OHL v.1.2 for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"
